File: Mk3/kicad/stm32l053c.kicad_pcb (KiCad board)
At the start: 2 copper layers, 26.7 x 43.2 mm, 45 parts, among them J1 GND, J10 3V3, J11 I2C, J2 GND, J3 TX, J4 GND, J5 TEST_1P, J6 TEST_1P, J8 RX, P1 SWD, U1 AP2112, U2 STM32L053C8_LQFP48, U3 ADS1015, U4 UFL_SMA, U5 RFM92/95

Commit message: Tweak traces
Routing:
- net Earth: track 219.6 -> 210.2 mm
- net /BATT: track 59.2 -> 54.0 mm, vias 3 -> 1
Changed lines of the file:
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@@
     (thickness 1.6)
     (drawings 66)
-    (tracks 521)
+    (tracks 511)
     (zones 0)
     (modules 45)
@@
     (effects (font (size 0.8 0.8) (thickness 0.15)))
   )
+  (segment (start 161.29 83.82) (end 159.93 83.82) (width 0.254) (layer F.Cu) (net 1))
+  (segment (start 159.93 83.82) (end 159.7 84.05) (width 0.254) (layer F.Cu) (net 1))
+  (segment (start 159.7 84.05) (end 159.7 91.425) (width 0.254) (layer F.Cu) (net 1))
+  (segment (start 159.7 91.425) (end 161.275 91.425) (width 0.254) (layer F.Cu) (net 1))
+  (segment (start 161.275 91.425) (end 161.29 91.44) (width 0.254) (layer F.Cu) (net 1))
   (segment (start 159.15 80.936185) (end 159.15 81.475) (width 0.254) (layer B.Cu) (net 1))
   (segment (start 157.099994 72.5) (end 159.15 74.550006) (width 0.254) (layer B.Cu) (net 1))
@@
   (segment (start 159.15 74.550006) (end 159.15 80.936185) (width 0.254) (layer B.Cu) (net 1))
   (via (at 159.15 81.475) (size 0.762) (drill 0.4064) (layers F.Cu B.Cu) (net 1))
-  (segment (start 161.29 83.82) (end 159.7 85.41) (width 0.254) (layer F.Cu) (net 1))
-  (segment (start 159.7 85.41) (end 159.7 89.85) (width 0.254) (layer F.Cu) (net 1))
-  (segment (start 159.7 89.85) (end 160.440001 90.590001) (width 0.254) (layer F.Cu) (net 1))
-  (segment (start 160.440001 90.590001) (end 161.29 91.44) (width 0.254) (layer F.Cu) (net 1))
   (segment (start 151.1 87.825) (end 148.674996 87.825) (width 0.254) (layer F.Cu) (net 1))
   (segment (start 148.674996 87.825) (end 145.499996 91) (width 0.254) (layer F.Cu) (net 1))
@@
   (segment (start 155.8 59.65) (end 155.95 59.5) (width 0.254) (layer B.Cu) (net 1))
   (segment (start 155.95 59.5) (end 159.57 55.88) (width 0.254) (layer B.Cu) (net 1))
-  (segment (start 152.2 59.7) (end 155.75 59.7) (width 0.254) (layer B.Cu) (net 1))
   (segment (start 155.75 59.7) (end 155.95 59.5) (width 0.254) (layer B.Cu) (net 1))
   (segment (start 145.97 63.246) (end 146.07 63.246) (width 0.254) (layer B.Cu) (net 1))
-  (segment (start 146.07 63.246) (end 148.804799 60.511201) (width 0.254) (layer B.Cu) (net 1))
-  (segment (start 148.804799 60.511201) (end 150.541377 60.511201) (width 0.254) (layer B.Cu) (net 1))
-  (segment (start 150.541377 60.511201) (end 150.563779 60.488799) (width 0.254) (layer B.Cu) (net 1))
-  (segment (start 150.563779 60.488799) (end 151.411201 60.488799) (width 0.254) (layer B.Cu) (net 1))
-  (segment (start 151.411201 60.488799) (end 152.2 59.7) (width 0.254) (layer B.Cu) (net 1))
   (segment (start 140.3 68.138815) (end 140.3 67.6) (width 0.254) (layer B.Cu) (net 1))
   (segment (start 140.3 70.774) (end 140.3 68.138815) (width 0.254) (layer B.Cu) (net 1))
@@
   (segment (start 137.16 81.28) (end 138.557 81.28) (width 0.254) (layer B.Cu) (net 38))
   (segment (start 138.557 81.28) (end 139.319 80.518) (width 0.254) (layer B.Cu) (net 38))
-  (segment (start 138.1 69.2) (end 138.1 63.2) (width 0.254) (layer B.Cu) (net 49))
-  (segment (start 150.9 59.3) (end 150.6 59.3) (width 0.254) (layer F.Cu) (net 49))
-  (segment (start 138.1 63.2) (end 142.380999 58.919001) (width 0.254) (layer B.Cu) (net 49))
-  (segment (start 152.8 61.2) (end 150.9 59.3) (width 0.254) (layer F.Cu) (net 49))
-  (segment (start 150.219001 58.919001) (end 150.6 59.3) (width 0.254) (layer B.Cu) (net 49))
-  (segment (start 142.380999 58.919001) (end 150.219001 58.919001) (width 0.254) (layer B.Cu) (net 49))
-  (via (at 150.6 59.3) (size 0.762) (drill 0.4064) (layers F.Cu B.Cu) (net 49))
-  (segment (start 152.8 61.2) (end 152.8 61.85) (width 0.254) (layer B.Cu) (net 49))
-  (segment (start 152.8 61.85) (end 154.15 63.2) (width 0.254) (layer B.Cu) (net 49))
+  (segment (start 138.1 69.2) (end 138.125 69.175) (width 0.254) (layer B.Cu) (net 49))
+  (segment (start 138.125 69.175) (end 138.125 68.375) (width 0.254) (layer B.Cu) (net 49))
+  (segment (start 138.125 68.375) (end 145.425 61.075) (width 0.254) (layer B.Cu) (net 49))
+  (segment (start 145.425 61.075) (end 152.025 61.075) (width 0.254) (layer B.Cu) (net 49))
   (segment (start 154.15 63.2) (end 154.25 63.2) (width 0.254) (layer B.Cu) (net 49))
-  (via (at 152.8 61.2) (size 0.762) (drill 0.4064) (layers F.Cu B.Cu) (net 49))
+  (segment (start 152.025 61.075) (end 154.15 63.2) (width 0.254) (layer B.Cu) (net 49))
   (segment (start 138.7 86.256) (end 138.7 69.8) (width 0.254) (layer F.Cu) (net 49))
   (segment (start 138.7 69.8) (end 138.1 69.2) (width 0.254) (layer F.Cu) (net 49))
